File: joystick-pcb/joystic-rj45.kicad_pcb (KiCad board)
At the start: 2 copper layers, 38 x 22 mm, 7 parts, among them CN1 1x5, CN2 1x8, CN3 1x2, CN4 1x2

Commit message: added commodore adapter pcb to this project. created gerbers
Other:
- net class Default removed
