File: commodore-adapter/commodore-adapter.kicad_sch (KiCad schematic)
At the start: 2 parts, among them CN1 1x9, CN2 1x8

Commit message: fixed DB9 pinout from male to female
Parts:
- CN1: footprint d-sub:DB9 board edge -> d-sub:DB9 female board edge
Changed lines of the file:
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@@
 			)
 		)
-		(property "Footprint" "d-sub:DB9 board edge"
+		(property "Footprint" "d-sub:DB9 female board edge"
 			(at 152.4 91.44 0)
 			(effects
